Commit message: completed moble manipulator without camera

File: gripper_car_ws/src/arm/arm_description/urdf/arm.urdf.xacro (robot description, xacro)
@@ -206,5 +206,5 @@
                         xyz="0.038 -0.024999 -0.00021816"
                         rpy="0.0087077 0.00057486 -0.06592"
-                        axis="0 0 -1"
+                        axis="0 0 1"
                         lower="-1.0" upper="0"
                         effort="2" velocity="1.0"
@@ -222,5 +222,5 @@
                         xyz="0.058 -0.016986 -0.0016533"
                         rpy="0.0087164 0.00042202 -0.048378"
-                        axis="0 0 -1"
+                        axis="0 0 1"
                         lower="-1.0" upper="0"
                         effort="2" velocity="1.0"

File: gripper_car_ws/src/arm/arm_description/urdf/arm_macro.urdf.xacro (robot description, xacro)
@@ -5,5 +5,11 @@
 -->
 <robot xmlns:xacro="http://www.ros.org/wiki/xacro">
-  <xacro:macro name="arm_macro" params="prefix parent *origin">
+ <!-- ================= ARM MACRO ================= -->
+  <xacro:macro name="arm_macro" params="parent prefix xyz rpy">
+    <joint name="${prefix}arm_base_joint" type="fixed">
+      <parent link="${parent}"/>
+      <child link="${prefix}base_link"/>
+      <origin xyz="${xyz}" rpy="${rpy}"/>
+    </joint>
     <!-- Inertia Macros -->
     <xacro:macro name="cyl_inertia" params="m r h">
@@ -17,15 +23,9 @@
                izz="${m*(x*x+y*y)/12.0}"/>
     </xacro:macro>
-    <!-- Base Joint -->
-    <joint name="${prefix}arm_base_joint" type="fixed">
-      <xacro:insert_block name="origin"/>
-      <parent link="${parent}"/>
-      <child link="${prefix}base_link"/>
-    </joint>
     <!-- Base Link -->
     <link name="${prefix}base_link">
       <visual>
         <geometry>
-          <mesh filename="package://arm_description/meshes/arm_base_link.STL"/>
+          <mesh filename="package://arm_description/meshes/base_link.STL"/>
         </geometry>
         <material name="arm_mat"><color rgba="0.8 0.8 0.9 1.0"/></material>
@@ -33,5 +33,5 @@
       <collision>
         <geometry>
-          <mesh filename="package://arm_description/meshes/arm_base_link.STL"/>
+          <mesh filename="package://arm_description/meshes/base_link.STL"/>
         </geometry>
       </collision>
@@ -91,5 +91,5 @@
       <parent link="${prefix}link_2"/>
       <child link="${prefix}link_3"/>
-      <axis xyz="0 1 0"/>
+      <axis xyz="0.0012899 -0.99996 -0.0086307"/>  <!-- CORRECTED -->
       <limit lower="${-pi/2}" upper="${pi/2}" effort="10.0" velocity="2.0"/>
     </joint>
@@ -113,5 +113,5 @@
       <parent link="${prefix}link_3"/>
       <child link="${prefix}link_4"/>
-      <axis xyz="0 1 0"/>
+      <axis xyz="0.99996 0.0002412 -0.0091073"/>  <!-- CORRECTED -->
       <limit lower="${-pi/2}" upper="${pi/2}" effort="5.0" velocity="2.0"/>
     </joint>
@@ -135,5 +135,5 @@
       <parent link="${prefix}link_4"/>
       <child link="${prefix}gripper_base_link"/>
-      <axis xyz="0 0 1"/>
+      <axis xyz="0 0.99996 0.0087265"/>  <!-- CORRECTED -->
       <limit lower="${-pi}" upper="${pi}" effort="5.0" velocity="2.0"/>
     </joint>
@@ -157,6 +157,6 @@
       <parent link="${prefix}gripper_base_link"/>
       <child link="${prefix}left_gear_link"/>
-      <axis xyz="0 1 0"/>
-      <limit lower="0" upper="${pi/4}" effort="5.0" velocity="1.0"/>
+      <axis xyz="0 0 1"/>  <!-- CORRECTED -->
+      <limit lower="0" upper="1.0" effort="5.0" velocity="1.0"/>  <!-- CORRECTED upper limit -->
     </joint>
     <link name="${prefix}left_gear_link">
@@ -175,8 +175,11 @@
     </link>
     <!-- Left Link + Finger (simplified) -->
-    <joint name="${prefix}left_link_joint" type="fixed">
+    <joint name="${prefix}left_joint" type="revolute">
       <origin xyz="0.058 -0.016986 -0.0016533" rpy="0.0087164 0.00042202 -0.048378"/>
-      <parent link="${prefix}left_gear_link"/>
+      <parent link="${prefix}gripper_base_link"/>
       <child link="${prefix}left_link"/>
+      <axis xyz="0 0 1"/>
+      <limit lower="-1.0" upper="0" effort="2" velocity="1.0"/>
+      <mimic joint="${prefix}left_gear_joint" multiplier="-1" offset="0"/>
     </joint>
     <link name="${prefix}left_link">
@@ -189,8 +192,11 @@
       </inertial>
     </link>
-    <joint name="${prefix}left_finger_joint" type="fixed">
+    <joint name="${prefix}left_finger_joint" type="revolute">
       <origin xyz="0.030728 0.0010745 0.013997" rpy="0 0 -0.4368"/>
-      <parent link="${prefix}left_link"/>
+      <parent link="${prefix}left_gear_link"/>
       <child link="${prefix}left_finger_link"/>
+      <axis xyz="0 0 -1"/>
+      <limit lower="0" upper="1.0" effort="2" velocity="1.0"/>
+      <mimic joint="${prefix}left_gear_joint" multiplier="1" offset="0"/>
     </joint>
     <link name="${prefix}left_finger_link">
@@ -208,6 +214,6 @@
       <parent link="${prefix}gripper_base_link"/>
       <child link="${prefix}right_gear_link"/>
-      <axis xyz="0 1 0"/>
-      <limit lower="${-pi/4}" upper="0" effort="5.0" velocity="1.0"/>
+      <axis xyz="0 0 1"/>  <!-- CORRECTED -->
+      <limit lower="-1.0" upper="0" effort="5.0" velocity="1.0"/>  <!-- CORRECTED lower limit -->
       <mimic joint="${prefix}left_gear_joint" multiplier="-1" offset="0"/>
     </joint>
@@ -222,8 +228,11 @@
     </link>
     <!-- Right Link + Finger -->
-    <joint name="${prefix}right_link_joint" type="fixed">
+    <joint name="${prefix}right_joint" type="revolute">
       <origin xyz="0.058 -0.0069838 -0.001891" rpy="0.0087015 -0.00066156 0.07588"/>
-      <parent link="${prefix}right_gear_link"/>
+      <parent link="${prefix}gripper_base_link"/>
       <child link="${prefix}right_link"/>
+      <axis xyz="0 0 1"/>
+      <limit lower="0" upper="1.0" effort="2" velocity="1.0"/>
+      <mimic joint="${prefix}left_gear_joint" multiplier="1" offset="0"/>
     </joint>
     <link name="${prefix}right_link">
@@ -236,8 +245,11 @@
       </inertial>
     </link>
-    <joint name="${prefix}right_finger_joint" type="fixed">
+    <joint name="${prefix}right_finger_joint" type="revolute">
       <origin xyz="0.030747 0 0.0055031" rpy="-3.1416 0 0.46391"/>
-      <parent link="${prefix}right_link"/>
+      <parent link="${prefix}right_gear_link"/>
       <child link="${prefix}right_finger_link"/>
+      <axis xyz="0 0 -1"/>
+      <limit lower="0" upper="1.0" effort="2" velocity="1.0"/>
+      <mimic joint="${prefix}left_gear_joint" multiplier="1" offset="0"/>
     </joint>
     <link name="${prefix}right_finger_link">
@@ -250,4 +262,5 @@
       </inertial>
     </link>
+    <!-- ADD MISSING MIMIC JOINTS -->
   </xacro:macro>
 </robot>

File: gripper_car_ws/src/mobile_base/mobile_base_description/urdf/mobile_base.urdf.xacro (robot description, xacro)
@@ -104,40 +104,9 @@
   <xacro:wheel name="back_right" reflect_y="-1" reflect_x="-1"/>
   <xacro:wheel name="back_left" reflect_y="1" reflect_x="-1"/>
-  <!-- LiDAR -->
-  <joint name="lidar_joint" type="fixed">
-    <parent link="body_link"/>
-    <child link="lidar_link"/>
-    <origin xyz="-0.15 0 ${chassis_height/2 + lidar_height/2}" rpy="0 0 0"/>
-  </joint>
-  <link name="lidar_link">
-    <visual>
-      <geometry>
-        <cylinder radius="${lidar_radius}" length="${lidar_height}"/>
-      </geometry>
-      <material name="lidar_black">
-        <color rgba="0.1 0.1 0.1 1.0"/>
-      </material>
-    </visual>
-    <collision>
-      <geometry>
-        <cylinder radius="${lidar_radius}" length="${lidar_height}"/>
-      </geometry>
-    </collision>
-    <inertial>
-      <mass value="${lidar_mass}"/>
-      <xacro:cylinder_inertia m="${lidar_mass}" r="${lidar_radius}" h="${lidar_height}"/>
-    </inertial>
-  </link>
-  <joint name="laser_frame_joint" type="fixed">
-    <parent link="lidar_link"/>
-    <child link="laser_frame"/>
-    <origin xyz="0 0 0" rpy="0 0 0"/>
-  </joint>
-  <link name="laser_frame"/>
   <!-- Camera -->
   <joint name="camera_joint" type="fixed">
     <parent link="body_link"/>
     <child link="camera_link"/>
-    <origin xyz="${chassis_length/2 + camera_depth/2} 0 ${chassis_height/2 - 0.02}" rpy="0 0 0"/>
+    <origin xyz="-${chassis_length/2 + camera_depth/2} 0 ${chassis_height/2 - 0.02}" rpy="0 0 0"/>
   </joint>
   <link name="camera_link">
